File: controller/thermoamp.kicad_sch (KiCad schematic)
At the start: 24 parts, among them J5 Conn_01x02_Socket, J6 Conn_01x02_Socket, U1 NJM4556A, U2 NJM4556A

Commit message: Updated schematic for thermo couple amp
Parts:
- removed R2_A2: 10k, Resistor_THT:R_Axial_DIN0207_L6.3mm_D2.5mm_P10.16mm_Horizontal, symbol Device:R_US
- removed RF_A2: 15k, Resistor_THT:R_Axial_DIN0207_L6.3mm_D2.5mm_P10.16mm_Horizontal, symbol Device:R_US
- added R1_B2: 1k, Resistor_THT:R_Axial_DIN0207_L6.3mm_D2.5mm_P10.16mm_Horizontal, symbol Device:R_US
- R1_B1: value 1.2k -> 180R
- R2_A1: value 220k -> 12k
- RF_A1: value 100k -> 12k
- RF_B1: value 180k -> 220k
- RF_B2: value 18k -> 150k
- RG_B1: value 18k -> 4.7k
Connections:
- net +12V: now also R1_B2.1
- net at R2_A1.2: now also R1_A1.2, U1.5 (+)
- net at C5.1, R2_A1.1, U1.1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: no longer R1_B1.1
- net at RL_A1.2, U1.7, U2.3 (+): now also RF_A1.2
- new net: R1_B1.1, R1_B2.2
Changed lines of the file:
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@@
   (junction (at 76.2 67.31) (diameter 0) (color 0 0 0 0)
   )
+  (junction (at 109.22 50.8) (diameter 0) (color 0 0 0 0)
+  )
   (junction (at 163.83 27.94) (diameter 0) (color 0 0 0 0)
   )
   (junction (at 41.91 130.81) (diameter 0) (color 0 0 0 0)
-  )
-  (junction (at 109.22 50.8) (diameter 0) (color 0 0 0 0)
   )
   (junction (at 144.78 53.34) (diameter 0) (color 0 0 0 0)
@@
   (no_connect (at 182.88 130.81))
   (no_connect (at 198.12 133.35))
+  (wire (pts (xy 129.54 20.32) (xy 129.54 27.94))
+    (stroke (width 0) (type default))
+  )
   (wire (pts (xy 189.23 48.26) (xy 181.61 48.26))
     (stroke (width 0) (type default))
@@
     (stroke (width 0) (type default))
   )
-  (wire (pts (xy 144.78 67.31) (xy 144.78 72.39))
-    (stroke (width 0) (type default))
-  )
   (wire (pts (xy 99.06 76.2) (xy 109.22 76.2))
     (stroke (width 0) (type default))
   )
+  (wire (pts (xy 144.78 27.94) (xy 151.13 27.94))
+    (stroke (width 0) (type default))
+  )
   (wire (pts (xy 135.89 72.39) (xy 144.78 72.39))
     (stroke (width 0) (type default))
@@
     (stroke (width 0) (type default))
   )
-  (wire (pts (xy 76.2 27.94) (xy 151.13 27.94))
-    (stroke (width 0) (type default))
-  )
-  (wire (pts (xy 76.2 50.8) (xy 76.2 27.94))
-    (stroke (width 0) (type default))
-  )
   (wire (pts (xy 109.22 71.12) (xy 109.22 73.66))
     (stroke (width 0) (type default))
@@
     (stroke (width 0) (type default))
   )
-  (wire (pts (xy 90.17 50.8) (xy 93.98 50.8))
+  (wire (pts (xy 90.17 50.8) (xy 109.22 50.8))
     (stroke (width 0) (type default))
   )
@@
     (stroke (width 0) (type default))
   )
+  (wire (pts (xy 129.54 27.94) (xy 137.16 27.94))
+    (stroke (width 0) (type default))
+  )
   (wire (pts (xy 109.22 50.8) (xy 109.22 63.5))
     (stroke (width 0) (type default))
@@
     (stroke (width 0) (type default))
   )
-  (wire (pts (xy 144.78 53.34) (xy 144.78 59.69))
+  (wire (pts (xy 144.78 53.34) (xy 144.78 72.39))
     (stroke (width 0) (type default))
   )
@@
   )
   (wire (pts (xy 76.2 67.31) (xy 76.2 77.47))
-    (stroke (width 0) (type default))
-  )
-  (wire (pts (xy 101.6 50.8) (xy 109.22 50.8))
     (stroke (width 0) (type default))
   )
@@
         (path "/12246f82-5c9a-456f-a9a1-28ea473855be/af061c45-1919-4b2b-92a8-7101c6ea2583"
           (reference "RL_B1") (unit 1)
-        )
-      )
-    )
-  )
-  (symbol (lib_id "Device:R_US") (at 97.79 50.8 90) (unit 1)
-    (in_bom yes) (on_board yes) (dnp no) (fields_autoplaced)
-    (property "Reference" "R2_A2" (at 97.79 44.45 90)
-      (effects (font (size 1.27 1.27)))
-    )
-    (property "Value" "10k" (at 97.79 46.99 90)
-      (effects (font (size 1.27 1.27)))
-    )
-    (property "Footprint" "Resistor_THT:R_Axial_DIN0207_L6.3mm_D2.5mm_P10.16mm_Horizontal" (at 98.044 49.784 90)
-      (effects (font (size 1.27 1.27)) hide)
-    )
-    (property "Datasheet" "~" (at 97.79 50.8 0)
-      (effects (font (size 1.27 1.27)) hide)
-    )
-    (pin "1")
-    (pin "2")
-    (instances
-      (project "controller"
-        (path "/12246f82-5c9a-456f-a9a1-28ea473855be/af061c45-1919-4b2b-92a8-7101c6ea2583"
-          (reference "R2_A2") (unit 1)
         )
       )
@@
     )
   )
+  (symbol (lib_id "power:+12V") (at 129.54 20.32 0) (unit 1)
+    (in_bom yes) (on_board yes) (dnp no) (fields_autoplaced)
+    (property "Reference" "#PWR033" (at 129.54 24.13 0)
+      (effects (font (size 1.27 1.27)) hide)
+    )
+    (property "Value" "+12V" (at 129.54 15.24 0)
+      (effects (font (size 1.27 1.27)))
+    )
+    (property "Footprint" "" (at 129.54 20.32 0)
+      (effects (font (size 1.27 1.27)) hide)
+    )
+    (property "Datasheet" "" (at 129.54 20.32 0)
+      (effects (font (size 1.27 1.27)) hide)
+    )
+    (pin "1")
+    (instances
+      (project "controller"
+        (path "/12246f82-5c9a-456f-a9a1-28ea473855be/af061c45-1919-4b2b-92a8-7101c6ea2583"
+          (reference "#PWR033") (unit 1)
+        )
+      )
+    )
+  )
   (symbol (lib_id "Connector:Conn_01x02_Socket") (at 123.19 127 0) (unit 1)
     (in_bom yes) (on_board yes) (dnp no) (fields_autoplaced)
@@
       (effects (font (size 1.27 1.27)))
     )
-    (property "Value" "1.2k" (at 154.94 24.13 90)
+    (property "Value" "180R" (at 154.94 24.13 90)
       (effects (font (size 1.27 1.27)))
     )
@@
       (effects (font (size 1.27 1.27)))
     )
-    (property "Value" "18k" (at 172.72 24.13 90)
+    (property "Value" "4.7k" (at 172.72 24.13 90)
       (effects (font (size 1.27 1.27)))
     )
@@
       (effects (font (size 1.27 1.27)))
     )
-    (property "Value" "220k" (at 86.36 46.99 90)
+    (property "Value" "12k" (at 86.36 46.99 90)
       (effects (font (size 1.27 1.27)))
     )
@@
       (effects (font (size 1.27 1.27)))
     )
-    (property "Value" "18k" (at 217.17 24.13 90)
+    (property "Value" "150k" (at 217.17 24.13 90)
       (effects (font (size 1.27 1.27)))
     )
@@
       (effects (font (size 1.27 1.27)))
     )
-    (property "Value" "180k" (at 203.2 24.13 90)
+    (property "Value" "220k" (at 203.2 24.13 90)
       (effects (font (size 1.27 1.27)))
     )
@@
         (path "/12246f82-5c9a-456f-a9a1-28ea473855be/af061c45-1919-4b2b-92a8-7101c6ea2583"
           (reference "C3") (unit 1)
+        )
+      )
+    )
+  )
+  (symbol (lib_id "Device:R_US") (at 140.97 27.94 90) (unit 1)
+    (in_bom yes) (on_board yes) (dnp no) (fields_autoplaced)
+    (property "Reference" "R1_B2" (at 140.97 21.59 90)
+      (effects (font (size 1.27 1.27)))
+    )
+    (property "Value" "1k" (at 140.97 24.13 90)
+      (effects (font (size 1.27 1.27)))
+    )
+    (property "Footprint" "Resistor_THT:R_Axial_DIN0207_L6.3mm_D2.5mm_P10.16mm_Horizontal" (at 141.224 26.924 90)
+      (effects (font (size 1.27 1.27)) hide)
+    )
+    (property "Datasheet" "~" (at 140.97 27.94 0)
+      (effects (font (size 1.27 1.27)) hide)
+    )
+    (pin "1")
+    (pin "2")
+    (instances
+      (project "controller"
+        (path "/12246f82-5c9a-456f-a9a1-28ea473855be/af061c45-1919-4b2b-92a8-7101c6ea2583"
+          (reference "R1_B2") (unit 1)
         )
       )
@@
     )
   )
-  (symbol (lib_id "Device:R_US") (at 144.78 63.5 0) (unit 1)
-    (in_bom yes) (on_board yes) (dnp no) (fields_autoplaced)
-    (property "Reference" "RF_A2" (at 147.32 62.23 0)
-      (effects (font (size 1.27 1.27)) (justify left))
-    )
-    (property "Value" "15k" (at 147.32 64.77 0)
-      (effects (font (size 1.27 1.27)) (justify left))
-    )
-    (property "Footprint" "Resistor_THT:R_Axial_DIN0207_L6.3mm_D2.5mm_P10.16mm_Horizontal" (at 145.796 63.754 90)
-      (effects (font (size 1.27 1.27)) hide)
-    )
-    (property "Datasheet" "~" (at 144.78 63.5 0)
-      (effects (font (size 1.27 1.27)) hide)
-    )
-    (pin "1")
-    (pin "2")
-    (instances
-      (project "controller"
-        (path "/12246f82-5c9a-456f-a9a1-28ea473855be/af061c45-1919-4b2b-92a8-7101c6ea2583"
-          (reference "RF_A2") (unit 1)
-        )
-      )
-    )
-  )
   (symbol (lib_id "Amplifier_Operational:NJM4556A") (at 60.96 67.31 0) (mirror x) (unit 1)
     (in_bom yes) (on_board yes) (dnp no)
@@
       (effects (font (size 1.27 1.27)))
     )
-    (property "Value" "100k" (at 132.08 68.58 90)
-      (effects (font (size 1.27 1.27)))
-    )
+    (property "Value" "12k" (at 132.08 68.58 90)
+      (effects (font (size 1.27 1.27)))
+    )

Commit message: Updated schematic
Parts:
- removed C4, C5: 100n, Capacitor_THT:C_Disc_D5.0mm_W2.5mm_P2.50mm, symbol Device:C
- removed R1_B1: 180R, Resistor_THT:R_Axial_DIN0207_L6.3mm_D2.5mm_P10.16mm_Horizontal, symbol Device:R_US
- removed R7: 4.7k, Resistor_THT:R_Axial_DIN0207_L6.3mm_D2.5mm_P10.16mm_Horizontal, symbol Device:R_US
- removed RF_B2: 150k, Resistor_THT:R_Axial_DIN0207_L6.3mm_D2.5mm_P10.16mm_Horizontal, symbol Device:R_US
- removed RL_B1: 10k, Resistor_THT:R_Axial_DIN0207_L6.3mm_D2.5mm_P10.16mm_Horizontal, symbol Device:R_US
- removed U2: NJM4556A, Package_SO:TSSOP-8_4.4x3mm_P0.65mm, symbol Amplifier_Operational:NJM4556A
- added RF_A2: 1k, Resistor_THT:R_Axial_DIN0207_L6.3mm_D2.5mm_P10.16mm_Horizontal, symbol Device:R_US
- R1_B1: renamed from R1_B2; value 1k -> 560R
- R2_A1: value 12k -> 22k
- R6: value 4.7k -> 1Meg
- RF_B1: value 220k -> 100k
- Rdown1: value 4.7k -> 18k
- renumbered J6 to J5, J5 to J6
Connections:
- net +12V: now also R2_A1.1; no longer R6.1
- net GND: now also R6.1
- net at Rup1.2: now also RF_B1.2, U1.7
- net at R1_A1.2, R2_A1.2: now also R6.2, U1.3 (+); no longer U1.5 (+)
- net at R1_B1.2: now also R2_B1.2, RG_B1.1
- net at RF_A1.1, RG_A1.2: now also U1.2 (-); no longer U1.6 (-)
- net at RF_B1.1, RG_B1.2: now also U1.6 (-)
- new net: RF_A1.2, RF_A2.1
- new net: RF_A2.2, RL_A1.2, U1.1, U1.5 (+)
- no-connect marks 3 -> 0
Other:
- moved on the sheet: J5, R1_A1, U1A, U1B

Commit message: Changed voltage divider values to ensure 3.3V limit on Tiva
Parts:
- Rdown1: value 18k -> 6.8k
- Rup1: value 8.2k -> 18k
Changed lines of the file:
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@@
       (effects (font (size 1.27 1.27)) (justify right))
     )
-    (property "Value" "8.2k" (at 228.6 64.77 0)
+    (property "Value" "18k" (at 228.6 64.77 0)
       (effects (font (size 1.27 1.27)) (justify right))
     )
@@
       (effects (font (size 1.27 1.27)) (justify right))
     )
-    (property "Value" "18k" (at 228.6 82.55 0)
+    (property "Value" "6.8k" (at 228.6 82.55 0)
       (effects (font (size 1.27 1.27)) (justify right))
     )
