File: tiva-board/tiva-board.kicad_pcb (KiCad board)
At the start: 2 copper layers, 100 x 100 mm, 28 parts, among them J1 Printstecker_1x03, J2 Printstecker_1x03, J3 Printstecker_1x02, J4 Printstecker_1x02, J5 Printstecker_1x02, J6 Printstecker_1x04, J7 Conn_01x04_Socket, U1 NJM4556A

Commit message: Extended documentation on Tiva board
Routing:
- net +3.3V: vias 0 -> 1
Changed lines of the file:
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@@
+    (effects (font (size 1 1) (thickness 0.15)) (justify left bottom))
+  )
+  (gr_text "SCL" (at 192.278 121.412 45) (layer "F.SilkS")
     (effects (font (size 1 1) (thickness 0.15)) (justify left bottom))
   )
@@
     (effects (font (size 1 1) (thickness 0.15)) (justify left bottom))
   )
+  (gr_text "+3.3V" (at 188.976 121.666 45) (layer "F.SilkS")
+    (effects (font (size 1 1) (thickness 0.15)) (justify left bottom))
+  )
   (gr_text "GND" (at 195.58 87.63) (layer "F.SilkS")
     (effects (font (size 1 1) (thickness 0.15)) (justify left bottom))
@@
     (effects (font (size 1 1) (thickness 0.15)) (justify left bottom))
   )
+  (gr_text "SDA" (at 195.072 121.412 45) (layer "F.SilkS")
+    (effects (font (size 1 1) (thickness 0.15)) (justify left bottom))
+  )
   (gr_text "3.9k" (at 119.38 76.2) (layer "F.SilkS")
     (effects (font (size 1 1) (thickness 0.15)) (justify left bottom))
   )
-  (gr_text "I2C connection and\npower supply for\nBMP280 temperature\nand pressure sensor" (at 196.85 133.35) (layer "F.SilkS")
+  (gr_text "I2C connection and\npower supply for\nBMP280 temperature\nand pressure sensor" (at 196.85 132.08) (layer "F.SilkS")
     (effects (font (size 1 1) (thickness 0.15)) (justify left bottom))
   )
@@
   )
   (gr_text "GND" (at 199.39 142.24) (layer "F.SilkS")
+    (effects (font (size 1 1) (thickness 0.15)) (justify left bottom))
+  )
+  (gr_text "GND" (at 186.69 121.412 45) (layer "F.SilkS")
     (effects (font (size 1 1) (thickness 0.15)) (justify left bottom))
   )
@@
     (style (thickness 0.15) (arrow_length 1.27) (text_position_mode 0) (extension_height 0.58642) (extension_offset 0.5) keep_text_aligned)
   )
-  (segment (start 189.23 120.65) (end 189.23 123.19) (width 0.25) (layer "F.Cu") (net 1))
   (segment (start 208.28 93.98) (end 200.66 86.36) (width 0.25) (layer "F.Cu") (net 1))
   (segment (start 208.28 110.49) (end 208.28 93.98) (width 0.25) (layer "F.Cu") (net 1))
-  (segment (start 205.74 113.03) (end 200.66 118.11) (width 0.25) (layer "F.Cu") (net 1))
   (segment (start 149.86 107.95) (end 146.05 104.14) (width 0.25) (layer "F.Cu") (net 1))
   (segment (start 152.4 137.16) (end 149.86 134.62) (width 0.25) (layer "F.Cu") (net 1))
   (segment (start 149.86 134.62) (end 149.86 107.95) (width 0.25) (layer "F.Cu") (net 1))
-  (segment (start 191.77 118.11) (end 189.23 120.65) (width 0.25) (layer "F.Cu") (net 1))
+  (segment (start 205.74 113.03) (end 201.93 116.84) (width 0.25) (layer "F.Cu") (net 1))
   (segment (start 186.69 137.16) (end 152.4 137.16) (width 0.25) (layer "F.Cu") (net 1))
   (segment (start 187.325 126.365) (end 187.325 132.08) (width 0.25) (layer "F.Cu") (net 1))
   (segment (start 205.74 113.03) (end 208.28 110.49) (width 0.25) (layer "F.Cu") (net 1))
   (segment (start 189.23 123.19) (end 189.23 124.46) (width 0.25) (layer "F.Cu") (net 1))
-  (segment (start 200.66 118.11) (end 191.77 118.11) (width 0.25) (layer "F.Cu") (net 1))
   (segment (start 128.494 105.186) (end 128.494 108.21) (width 0.25) (layer "F.Cu") (net 1))
   (segment (start 146.05 104.14) (end 129.54 104.14) (width 0.25) (layer "F.Cu") (net 1))
@@
   (segment (start 187.325 132.08) (end 187.325 136.525) (width 0.25) (layer "F.Cu") (net 1))
   (segment (start 187.325 136.525) (end 186.69 137.16) (width 0.25) (layer "F.Cu") (net 1))
+  (via (at 201.93 116.84) (size 0.8) (drill 0.4) (layers "F.Cu" "B.Cu") (net 1))
+  (segment (start 193.04 116.84) (end 189.23 120.65) (width 0.25) (layer "B.Cu") (net 1))
+  (segment (start 189.23 120.65) (end 189.23 123.19) (width 0.25) (layer "B.Cu") (net 1))
+  (segment (start 201.93 116.84) (end 193.04 116.84) (width 0.25) (layer "B.Cu") (net 1))
   (segment (start 149.86 92.71) (end 148.59 93.98) (width 0.25) (layer "F.Cu") (net 2))
   (segment (start 151.13 91.44) (end 149.86 92.71) (width 0.25) (layer "F.Cu") (net 2))
