File: tiva-board/tiva-board.kicad_pcb (KiCad board)
At the start: 2 copper layers, 100 x 100 mm, 28 parts, among them J1 Printstecker_1x03, J2 Printstecker_1x03, J3 Printstecker_1x02, J4 Printstecker_1x02, J5 Printstecker_1x02, J6 Printstecker_1x04, J7 Conn_01x04_Socket, U1 NJM4556A

Commit message: Updated resistor values on the Tiva board
Other:
- board text added: "1.0k"
- board text removed: "3.9k"
Changed lines of the file:
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@@
     (effects (font (size 1 1) (thickness 0.15)) (justify left bottom))
   )
-  (gr_text "3.9k" (at 167.64 57.15) (layer "F.SilkS")
+  (gr_text "1.0k" (at 167.64 57.15) (layer "F.SilkS")
     (effects (font (size 1 1) (thickness 0.15)) (justify left bottom))
   )
@@
     (effects (font (size 1 1) (thickness 0.15)) (justify left bottom))
   )
-  (gr_text "3.9k" (at 119.38 76.2) (layer "F.SilkS")
+  (gr_text "1.0k" (at 119.38 76.2) (layer "F.SilkS")
     (effects (font (size 1 1) (thickness 0.15)) (justify left bottom))
   )
