File: controller_v2/thermo_sensor.kicad_sch (KiCad schematic)
At the start: 15 parts, among them J10 Printstecker_1x03, J2 Conn_01x02_Pin, J5 Conn_01x02_Pin, J6 Printstecker_1x02, U1 max6675

Commit message: Cleanup schematic
Parts:
- removed J10: Printstecker_1x03, connectors:printstecker_1x03_P2.54mm, symbol connectors:printstecker_1x03
- removed J2, J5: Conn_01x02_Pin, Connector_PinSocket_2.54mm:PinSocket_1x02_P2.54mm_Vertical, symbol Connector:Conn_01x02_Pin
- removed TP1: TestPoint, TestPoint:TestPoint_THTPad_4.0x4.0mm_Drill2.0mm, symbol Connector:TestPoint
Changed lines of the file:
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@@
   (junction (at 113.03 120.65) (diameter 0) (color 0 0 0 0)
   )
-  (junction (at 143.51 120.65) (diameter 0) (color 0 0 0 0)
-  )
   (junction (at 113.03 138.43) (diameter 0) (color 0 0 0 0)
   )
   (junction (at 165.1 85.09) (diameter 0) (color 0 0 0 0)
   )
-  (junction (at 146.05 123.19) (diameter 0) (color 0 0 0 0)
-  )
   (junction (at 124.46 85.09) (diameter 0) (color 0 0 0 0)
   )
-  (wire (pts (xy 148.59 123.19) (xy 146.05 123.19))
-    (stroke (width 0) (type default))
-  )
   (wire (pts (xy 130.81 57.15) (xy 130.81 87.63))
     (stroke (width 0) (type default))
@@
     (stroke (width 0) (type default))
   )
-  (wire (pts (xy 165.1 85.09) (xy 193.04 85.09))
-    (stroke (width 0) (type default))
-  )
-  (wire (pts (xy 146.05 123.19) (xy 142.24 123.19))
+  (wire (pts (xy 165.1 85.09) (xy 191.77 85.09))
     (stroke (width 0) (type default))
   )
@@
     (stroke (width 0) (type default))
   )
-  (wire (pts (xy 113.03 138.43) (xy 142.24 138.43))
-    (stroke (width 0) (type default))
-  )
   (wire (pts (xy 124.46 85.09) (xy 142.24 85.09))
     (stroke (width 0) (type default))
   )
-  (wire (pts (xy 168.91 87.63) (xy 193.04 87.63))
+  (wire (pts (xy 168.91 87.63) (xy 195.58 87.63))
     (stroke (width 0) (type default))
   )
@@
     (stroke (width 0) (type default))
   )
-  (wire (pts (xy 69.85 128.27) (xy 69.85 135.89))
+  (wire (pts (xy 195.58 71.12) (xy 195.58 87.63))
     (stroke (width 0) (type default))
   )
@@
     (stroke (width 0) (type default))
   )
-  (wire (pts (xy 143.51 120.65) (xy 148.59 120.65))
-    (stroke (width 0) (type default))
-  )
   (wire (pts (xy 113.03 138.43) (xy 113.03 142.24))
     (stroke (width 0) (type default))
   )
-  (wire (pts (xy 148.59 114.3) (xy 146.05 114.3))
+  (wire (pts (xy 204.47 76.2) (xy 199.39 76.2))
     (stroke (width 0) (type default))
   )
@@
     (stroke (width 0) (type default))
   )
-  (wire (pts (xy 113.03 120.65) (xy 143.51 120.65))
-    (stroke (width 0) (type default))
-  )
   (wire (pts (xy 146.05 60.96) (xy 146.05 64.77))
     (stroke (width 0) (type default))
   )
+  (wire (pts (xy 199.39 76.2) (xy 199.39 90.17))
+    (stroke (width 0) (type default))
+  )
   (wire (pts (xy 93.98 138.43) (xy 113.03 138.43))
     (stroke (width 0) (type default))
   )
-  (wire (pts (xy 148.59 111.76) (xy 143.51 111.76))
-    (stroke (width 0) (type default))
-  )
   (wire (pts (xy 113.03 115.57) (xy 113.03 120.65))
     (stroke (width 0) (type default))
@@
     (stroke (width 0) (type default))
   )
-  (wire (pts (xy 143.51 111.76) (xy 143.51 120.65))
-    (stroke (width 0) (type default))
-  )
   (wire (pts (xy 110.49 87.63) (xy 130.81 87.63))
     (stroke (width 0) (type default))
   )
-  (wire (pts (xy 142.24 123.19) (xy 142.24 138.43))
-    (stroke (width 0) (type default))
-  )
   (wire (pts (xy 124.46 49.53) (xy 124.46 85.09))
     (stroke (width 0) (type default))
   )
-  (wire (pts (xy 172.72 90.17) (xy 193.04 90.17))
+  (wire (pts (xy 191.77 66.04) (xy 191.77 85.09))
+    (stroke (width 0) (type default))
+  )
+  (wire (pts (xy 204.47 71.12) (xy 195.58 71.12))
+    (stroke (width 0) (type default))
+  )
+  (wire (pts (xy 172.72 90.17) (xy 199.39 90.17))
     (stroke (width 0) (type default))
   )
@@
     (stroke (width 0) (type default))
   )
-  (wire (pts (xy 146.05 114.3) (xy 146.05 123.19))
+  (wire (pts (xy 204.47 66.04) (xy 191.77 66.04))
     (stroke (width 0) (type default))
   )
@@
   (label "T(-)" (at 133.35 85.09 0) (fields_autoplaced)
     (effects (font (size 1.27 1.27)) (justify left bottom))
+  )
+  (hierarchical_label "~{CS}" (shape bidirectional) (at 204.47 71.12 0) (fields_autoplaced)
+    (effects (font (size 1.27 1.27)) (justify left))
+  )
+  (hierarchical_label "SO" (shape bidirectional) (at 204.47 66.04 0) (fields_autoplaced)
+    (effects (font (size 1.27 1.27)) (justify left))
+  )
+  (hierarchical_label "SCK" (shape bidirectional) (at 204.47 76.2 0) (fields_autoplaced)
+    (effects (font (size 1.27 1.27)) (justify left))
   )
   (symbol (lib_id "active:max6675") (at 149.86 86.36 0) (unit 1)
@@
     )
   )
-  (symbol (lib_id "connectors:printstecker_1x03") (at 198.12 87.63 0) (unit 1)
-    (in_bom yes) (on_board yes) (dnp no) (fields_autoplaced)
-    (property "Reference" "J10" (at 199.39 86.36 0)
-      (effects (font (size 1.27 1.27)) (justify left))
-    )
-    (property "Value" "Printstecker_1x03" (at 199.39 88.9 0)
-      (effects (font (size 1.27 1.27)) (justify left))
-    )
-    (property "Footprint" "connectors:printstecker_1x03_P2.54mm" (at 195.58 96.52 0)
-      (effects (font (size 1.27 1.27)) hide)
-    )
-    (property "Datasheet" "" (at 195.58 87.63 0)
-      (effects (font (size 1.27 1.27)) hide)
-    )
-    (pin "1")
-    (pin "2")
-    (pin "3")
-    (instances
-      (project "controller_v2"
-        (path "/884d8f78-75d7-4449-b027-2ba1bd4eeac8/58d7af1d-7239-4ab5-80a2-fcd44c87ce49"
-          (reference "J10") (unit 1)
-        )
-      )
-    )
-  )
   (symbol (lib_id "Connector:TestPoint") (at 124.46 49.53 0) (unit 1)
     (in_bom yes) (on_board yes) (dnp no) (fields_autoplaced)
@@
     )
   )
-  (symbol (lib_id "Connector:TestPoint") (at 69.85 128.27 0) (unit 1)
-    (in_bom yes) (on_board yes) (dnp no) (fields_autoplaced)
-    (property "Reference" "TP1" (at 72.39 123.698 0)
-      (effects (font (size 1.27 1.27)) (justify left))
-    )
-    (property "Value" "TestPoint" (at 72.39 126.238 0)
-      (effects (font (size 1.27 1.27)) (justify left))
-    )
-    (property "Footprint" "TestPoint:TestPoint_THTPad_4.0x4.0mm_Drill2.0mm" (at 74.93 128.27 0)
-      (effects (font (size 1.27 1.27)) hide)
-    )
-    (property "Datasheet" "~" (at 74.93 128.27 0)
-      (effects (font (size 1.27 1.27)) hide)
-    )
-    (pin "1")
-    (instances
-      (project "thermo-sensor-digital"
-        (path "/19ef6a1d-1471-49aa-9d9c-b1c1cdf31a28"
-          (reference "TP1") (unit 1)
-        )
-      )
-      (project "controller_v2"
-        (path "/884d8f78-75d7-4449-b027-2ba1bd4eeac8/58d7af1d-7239-4ab5-80a2-fcd44c87ce49"
-          (reference "TP6") (unit 1)
-        )
-      )
-    )
-  )
   (symbol (lib_id "power:+3.3V") (at 88.9 83.82 0) (unit 1)
     (in_bom yes) (on_board yes) (dnp no) (fields_autoplaced)
@@
         (path "/884d8f78-75d7-4449-b027-2ba1bd4eeac8/58d7af1d-7239-4ab5-80a2-fcd44c87ce49"
           (reference "#PWR019") (unit 1)
-        )
-      )
-    )
-  )
-  (symbol (lib_id "power:GND") (at 69.85 135.89 0) (unit 1)
-    (in_bom yes) (on_board yes) (dnp no) (fields_autoplaced)
-    (property "Reference" "#PWR01" (at 69.85 142.24 0)
-      (effects (font (size 1.27 1.27)) hide)
-    )
-    (property "Value" "GND" (at 69.85 140.97 0)
-      (effects (font (size 1.27 1.27)))
-    )
-    (property "Footprint" "" (at 69.85 135.89 0)
-      (effects (font (size 1.27 1.27)) hide)
-    )
-    (property "Datasheet" "" (at 69.85 135.89 0)
-      (effects (font (size 1.27 1.27)) hide)
-    )
-    (pin "1")
-    (instances
-      (project "thermo-sensor-digital"
-        (path "/19ef6a1d-1471-49aa-9d9c-b1c1cdf31a28"
-          (reference "#PWR01") (unit 1)
-        )
-      )
-      (project "controller_v2"
-        (path "/884d8f78-75d7-4449-b027-2ba1bd4eeac8/58d7af1d-7239-4ab5-80a2-fcd44c87ce49"
-          (reference "#PWR018") (unit 1)
         )
       )
@@
         )
       )
-    )
-  )
-  (symbol (lib_id "Connector:Conn_01x02_Pin") (at 153.67 123.19 180) (unit 1)
-    (in_bom yes) (on_board yes) (dnp no) (fields_autoplaced)
-    (property "Reference" "J2" (at 154.94 120.65 0)
-      (effects (font (size 1.27 1.27)) (justify right))
-    )
-    (property "Value" "Conn_01x02_Pin" (at 154.94 123.19 0)
-      (effects (font (size 1.27 1.27)) (justify right))
-    )
-    (property "Footprint" "Connector_PinSocket_2.54mm:PinSocket_1x02_P2.54mm_Vertical" (at 153.67 123.19 0)
-      (effects (font (size 1.27 1.27)) hide)
-    )
-    (property "Datasheet" "~" (at 153.67 123.19 0)
-      (effects (font (size 1.27 1.27)) hide)
-    )
-    (pin "1")
-    (pin "2")
-    (instances
-      (project "thermo-sensor-digital"
-        (path "/19ef6a1d-1471-49aa-9d9c-b1c1cdf31a28"
-          (reference "J2") (unit 1)
-        )
-      )
-      (project "controller_v2"
-        (path "/884d8f78-75d7-4449-b027-2ba1bd4eeac8/58d7af1d-7239-4ab5-80a2-fcd44c87ce49"
-          (reference "J8") (unit 1)
-        )
-      )
-    )
-  )
-  (symbol (lib_id "Connector:Conn_01x02_Pin") (at 153.67 114.3 180) (unit 1)
-    (in_bom yes) (on_board yes) (dnp no) (fields_autoplaced)
-    (property "Reference" "J5" (at 154.94 111.76 0)
-      (effects (font (size 1.27 1.27)) (justify right))
-    )
-    (property "Value" "Conn_01x02_Pin" (at 154.94 114.3 0)
-      (effects (font (size 1.27 1.27)) (justify right))
-    )
-    (property "Footprint" "Connector_PinSocket_2.54mm:PinSocket_1x02_P2.54mm_Vertical" (at 153.67 114.3 0)
-      (effects (font (size 1.27 1.27)) hide)
-    )
-    (property "Datasheet" "~" (at 153.67 114.3 0)
-      (effects (font (size 1.27 1.27)) hide)
-    )
-    (pin "1")
-    (pin "2")
-    (instances
-      (project "thermo-sensor-digital"
-        (path "/19ef6a1d-1471-49aa-9d9c-b1c1cdf31a28"
-          (reference "J5") (unit 1)
-        )
-      )
-      (project "controller_v2"
-        (path "/884d8f78-75d7-4449-b027-2ba1bd4eeac8/58d7af1d-7239-4ab5-80a2-fcd44c87ce49"
-          (reference "J7") (unit 1)
-        )
-      )
